File: PCB PhEC/Tds_NonSmd_PRINT.brd (EAGLE design)
At the start: 194.3 x 107.6 mm, 61 parts, among them IC1 TL074P, IC2 TL062P, X10 227161-8, X2 BN35N61, X4 R141426, X5 R141426, X8 BN35N61, X9 227161-8

Commit message: ADD PCB READY TO PRINT
Routing:
- net AGND: track 278.2 -> 283.9 mm
Changed lines of the file:
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@@
 <layer number="25" name="tNames" color="7" fill="1" visible="yes" active="yes"/>
 <layer number="26" name="bNames" color="7" fill="1" visible="yes" active="yes"/>
-<layer number="27" name="tValues" color="7" fill="1" visible="yes" active="yes"/>
-<layer number="28" name="bValues" color="7" fill="1" visible="yes" active="yes"/>
+<layer number="27" name="tValues" color="7" fill="1" visible="no" active="yes"/>
+<layer number="28" name="bValues" color="7" fill="1" visible="no" active="yes"/>
 <layer number="29" name="tStop" color="7" fill="3" visible="no" active="yes"/>
 <layer number="30" name="bStop" color="7" fill="6" visible="no" active="yes"/>
@@
 <layer number="41" name="tRestrict" color="4" fill="10" visible="yes" active="yes"/>
 <layer number="42" name="bRestrict" color="1" fill="10" visible="yes" active="yes"/>
-<layer number="43" name="vRestrict" color="2" fill="10" visible="yes" active="yes"/>
+<layer number="43" name="vRestrict" color="2" fill="10" visible="no" active="yes"/>
 <layer number="44" name="Drills" color="7" fill="1" visible="no" active="yes"/>
-<layer number="45" name="Holes" color="7" fill="1" visible="no" active="yes"/>
+<layer number="45" name="Holes" color="7" fill="1" visible="yes" active="yes"/>
 <layer number="46" name="Milling" color="3" fill="1" visible="no" active="yes"/>
 <layer number="47" name="Measures" color="7" fill="1" visible="no" active="yes"/>
-<layer number="48" name="Document" color="7" fill="1" visible="yes" active="yes"/>
-<layer number="49" name="Reference" color="7" fill="1" visible="yes" active="yes"/>
+<layer number="48" name="Document" color="7" fill="1" visible="no" active="yes"/>
+<layer number="49" name="Reference" color="7" fill="1" visible="no" active="yes"/>
 <layer number="51" name="tDocu" color="7" fill="1" visible="yes" active="yes"/>
 <layer number="52" name="bDocu" color="7" fill="1" visible="yes" active="yes"/>
@@
 <attribute name="MF" value="" x="-1.905" y="76.454" size="1.778" layer="27" rot="R90" display="off"/>
 <attribute name="MPN" value="" x="-1.905" y="76.454" size="1.778" layer="27" rot="R90" display="off"/>
-<attribute name="NAME" x="-6.35" y="66.3702" size="1.778" layer="25" ratio="10" rot="R90"/>
+<attribute name="NAME" x="-3.81" y="63.8302" size="1.778" layer="25" ratio="10" rot="R90"/>
 <attribute name="OC_FARNELL" value="unknown" x="-1.905" y="76.454" size="1.778" layer="27" rot="R90" display="off"/>
 <attribute name="OC_NEWARK" value="unknown" x="-1.905" y="76.454" size="1.778" layer="27" rot="R90" display="off"/>
@@
 <wire x1="39.37" y1="40.64" x2="38.1" y2="41.91" width="1.016" layer="16"/>
 <wire x1="38.1" y1="41.91" x2="35.56" y2="41.91" width="1.016" layer="16"/>
-<wire x1="49.53" y1="50.8" x2="49.53" y2="40.64" width="1.016" layer="16"/>
+<wire x1="49.53" y1="50.8" x2="49.53" y2="48.26" width="1.016" layer="16"/>
+<wire x1="49.53" y1="48.26" x2="49.53" y2="40.64" width="1.016" layer="16"/>
 <wire x1="44.45" y1="40.64" x2="39.37" y2="40.64" width="1.016" layer="16"/>
 <wire x1="35.56" y1="39.37" x2="35.56" y2="41.91" width="1.016" layer="16"/>
@@
 <wire x1="50.134540625" y1="80.040459375" x2="50.53" y2="80.43591875" width="1.27" layer="16"/>
 <wire x1="50.53" y1="80.43591875" x2="50.53" y2="81.534" width="1.27" layer="16"/>
+<wire x1="47.5488" y1="48.8188" x2="48.9712" y2="48.8188" width="1.27" layer="16"/>
+<wire x1="48.9712" y1="48.8188" x2="49.53" y2="48.26" width="1.27" layer="16"/>
+<wire x1="47.5488" y1="42.6212" x2="50.0888" y2="42.6212" width="1.27" layer="16"/>
+<wire x1="50.0888" y1="42.6212" x2="50.8" y2="41.91" width="1.27" layer="16"/>
 <wire x1="47.9298" y1="89.7128" x2="48.97708125" y2="89.043" width="0" layer="19" extent="16-16"/>
 </signal>

Commit message: UPDATE PCB NON SMD
Routing:
- net AGND: track 283.9 -> 273.5 mm
Changed lines of the file:
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@@
 <wire x1="-5.0546" y1="68.9356" x2="-5.08" y2="68.961" width="1.016" layer="16"/>
 <wire x1="-5.08" y1="35.56" x2="-3.81" y2="34.29" width="1.016" layer="16"/>
-<wire x1="-5.08" y1="58.674" x2="-5.08" y2="48.26" width="1.016" layer="16"/>
 <wire x1="-2.54" y1="48.26" x2="-5.08" y2="48.26" width="1.016" layer="16"/>
 <wire x1="8.382" y1="55.626" x2="6.096" y2="55.626" width="1.016" layer="16"/>
